Commit message: updated robot design

File: my_robot/urdf/my_robot.xacro (robot description, xacro)
@@ -1,170 +1,36 @@
+<?xml version='1.0'?>
 <robot name="my_robot" xmlns:xacro="http://www.ros.org/wiki/xacro">
-	<xacro:include filename="$(find my_robot)/urdf/my_robot.gazebo" />
-  <link name="robot_footprint"></link>
-  <joint name="robot_footprint_joint" type="fixed">
-    <origin xyz="0 0 0" rpy="0 0 0" />
-    <parent link="robot_footprint"/>
-    <child link="chassis" />
-  </joint>
-  <link name='chassis'>
-    <pose>0 0 0.1 0 0 0</pose>
-    <inertial>
-      <mass value="15.0"/>
-      <origin xyz="0.0 0 0" rpy=" 0 0 0"/>
-      <inertia
-          ixx="0.1" ixy="0" ixz="0"
-          iyy="0.1" iyz="0"
-          izz="0.1"
-      />
-    </inertial>
-    <collision name='collision'>
-      <origin xyz="0 0 0" rpy=" 0 0 0"/>
-      <geometry>
-        <cylinder length="0.1" radius="0.18"/>
-      </geometry>
-    </collision>
-    <visual name='chassis_visual'>
-      <origin xyz="0 0 0" rpy=" 0 0 0"/>
-      <geometry>
-        <cylinder length="0.1" radius="0.18"/>
-      </geometry>
-    </visual>
-		<!--spheres-->
-    <collision name='back_caster_collision'>
-      <origin xyz="-0.10 0 -0.05" rpy=" 0 0 0"/>
-      <geometry>
-        <sphere radius="0.045"/>
-      </geometry>
-    </collision>
-    <visual name='back_caster_visual'>
-      <origin xyz="-0.10 0 -0.05" rpy=" 0 0 0"/>
-      <geometry>
-        <sphere radius="0.045"/>
-      </geometry>
-    </visual>
-    <collision name='front_caster_collision'>
-      <origin xyz="0.10 0 -0.05" rpy=" 0 0 0"/>
-      <geometry>
-        <sphere radius="0.045"/>
-      </geometry>
-    </collision>
-    <visual name='front_caster_visual'>
-      <origin xyz="0.10 0 -0.05" rpy=" 0 0 0"/>
-      <geometry>
-        <sphere radius="0.045"/>
-      </geometry>
-    </visual>
-		<collision name='left_caster_collision'>
-      <origin xyz="0 -0.10 -0.05" rpy=" 0 0 0"/>
-      <geometry>
-        <sphere radius="0.045"/>
-      </geometry>
-    </collision>
-    <visual name='left_caster_visual'>
-      <origin xyz="0 -0.10 -0.05" rpy=" 0 0 0"/>
-      <geometry>
-        <sphere radius="0.045"/>
-      </geometry>
-    </visual>
-		<collision name='right_caster_collision'>
-      <origin xyz="0 0.10 -0.05" rpy=" 0 0 0"/>
-      <geometry>
-        <sphere radius="0.045"/>
-      </geometry>
-    </collision>
-    <visual name='right_caster_visual'>
-      <origin xyz="0 0.10 -0.05" rpy=" 0 0 0"/>
-      <geometry>
-        <sphere radius="0.045"/>
-      </geometry>
-    </visual>
-		<!--vertical tower-->
-		<collision name='tower_collision'>
-      <origin xyz="0 0 0.02" rpy="0 0 0"/>
-      <geometry>
-        <cylinder length="0.18" radius="0.03"/>
-      </geometry>
-    </collision>
-    <visual name='tower_visual'>
-      <origin xyz="0 0 0.02" rpy="0 0 0"/>
-      <geometry>
-        <cylinder length="0.18" radius="0.03"/>
-      </geometry>
-    </visual>
-		<!--horizontal rod 1-->
-		<collision name='rod_collision'>
-      <origin xyz="0 0 0" rpy="0 1.5707 1.5707"/>
-      <geometry>
-        <cylinder length="0.4" radius="0.03"/>
-      </geometry>
-    </collision>
-    <visual name='rod_visual'>
-      <origin xyz="0 0 0" rpy="0 1.5707 1.5707"/>
-      <geometry>
-        <cylinder length="0.4" radius="0.03"/>
-      </geometry>
-    </visual>
-  </link>
-	<!--horizontal additional mass-->
-		<link name='add_mass'>
-			<pose>0 0 0 0 0 0</pose>
-			<inertial>
-				<mass value="0.5"/>
-				<origin xyz="0.0 0 0" rpy="0 0 0"/>
-					<inertia
-						ixx="0.1" ixy="0" ixz="0"
-						iyy="0.1" iyz="0"
-						izz="0.1"
-					/>
-				</inertial>
-				<collision name='add_collision'>
-					<origin xyz="0 0 0" rpy="0 0 0"/>
-					<geometry>
-						<box size="0.05 0.05 0.05"/>
-					</geometry>
-				</collision>
-				<visual name='add_visual'>
-					<origin xyz="0 0 0" rpy="0 0 0"/>
-					<geometry>
-						<box size="0.05 0.05 0.05"/>
-					</geometry>
-				</visual>
-		</link>
-		<joint type="continuous" name="add_mass_hinge">
-			<origin xyz="-0.2 0 0" rpy="0 0 0"/>
-			<child link="add_mass"/>
-			<parent link="chassis"/>
-			<axis xyz="0 1 0" rpy="0 0 0"/>
-			<limit effort="10000" velocity="1000"/>
-			<dynamics damping="1.0" friction="1.0"/>
-		</joint>
-	<!--left wheel -->
-	<link name='left_wheel'>
-		<pose>0 0 0 0 0 0</pose>
-		<inertial>
-			<mass value="5.0"/>
-			<origin xyz="0.0 0 0" rpy=" 0 1.5707 1.5707"/>
-				<inertia
-					ixx="0.1" ixy="0" ixz="0"
-					iyy="0.1" iyz="0"
-					izz="0.1"
-				/>
-			</inertial>
-			<collision name='collision'>
-				<origin xyz="0 0 0" rpy=" 0 1.5707 1.5707"/>
-				<geometry>
-					<cylinder radius="0.1" length="0.06"/>
-				</geometry>
-			</collision>
-			<visual name='left_wheel_visual'>
-				<origin xyz="0 0 0" rpy=" 0 1.5707 1.5707"/>
-				<geometry>
-					<cylinder radius="0.1" length="0.06"/>
-				</geometry>
-			</visual>
-	</link>
-	<!--right wheel-->
-	<link name='right_wheel'>
-    <pose>0 0 0 0 0 0</pose>
+<xacro:include filename="$(find my_robot)/urdf/my_robot.gazebo" />
+<link name="robot_footprint"></link>
+<joint name="robot_footprint_joint" type="fixed">
+  <origin xyz="0 0 0" rpy="0 0 0" />
+  <parent link="robot_footprint"/>
+  <child link="chassis" />
+</joint>
+<link name='chassis'>
+  <pose>0 0 0.1 0 0 0</pose>
+  <inertial>
+    <mass value="15.0"/>
+    <origin xyz="0.0 0 0" rpy=" 0 0 0"/>
+    <inertia
+        ixx="0.1" ixy="0" ixz="0"
+        iyy="0.1" iyz="0"
+        izz="0.1"
+    />
+  </inertial>
+  <collision name='collision'>
+    <origin xyz="0 0 0" rpy=" 0 0 0"/>
+    <geometry>
+      <box size=".5 .3 .1"/>
+    </geometry>
+  </collision>
+  <visual name='chassis_visual'>
+    <origin xyz="0 0 0" rpy=" 0 0 0"/>
+    <geometry>
+      <box size=".5 .3 .1"/>
+    </geometry>
+  </visual>
+</link>
+<link name='left_wheel_front'>
     <inertial>
       <mass value="5.0"/>
@@ -176,115 +42,194 @@
       />
     </inertial>
-    <collision name='collision'>
+    <collision name='left_wheel_front_collision'>
       <origin xyz="0 0 0" rpy=" 0 1.5707 1.5707"/>
       <geometry>
-        <cylinder radius="0.1" length="0.06"/>
+        <cylinder radius=".08" length="0.044"/>
       </geometry>
     </collision>
-    <visual name='right_wheel_visual'>
+    <visual name='left_wheel_front_visual'>
       <origin xyz="0 0 0" rpy=" 0 1.5707 1.5707"/>
       <geometry>
-        <cylinder radius="0.1" length="0.06"/>
+        <cylinder radius=".08" length="0.044"/>
       </geometry>
     </visual>
   </link>
-	<!--left, right joint-->
-	<joint type="continuous" name="left_wheel_hinge">
-		<origin xyz="0 0.23 0" rpy="0 0 0"/>
-		<child link="left_wheel"/>
-		<parent link="chassis"/>
-		<axis xyz="0 1 0" rpy="0 0 0"/>
-		<limit effort="10000" velocity="1000"/>
-		<dynamics damping="1.0" friction="1.0"/>
-	</joint>
-	<joint type="continuous" name="right_wheel_hinge">
-    <origin xyz="0 -0.23 0" rpy="0 0 0"/>
-    <child link="right_wheel"/>
-    <parent link="chassis"/>
-    <axis xyz="0 1 0" rpy="0 0 0"/>
-    <limit effort="10000" velocity="1000"/>
-    <dynamics damping="1.0" friction="1.0"/>
-  </joint>
-	<!--camera-->
-	<link name='camera'>
-    <pose>0 0 0 0 0 0</pose>
-    <inertial>
-      <mass value="0.5"/>
-      <origin xyz="0.0 0 0" rpy="0.0 0 0"/>
-      <inertia
-          ixx="1e-6" ixy="0" ixz="0"
-          iyy="1e-6" iyz="0"
-          izz="1e-6"
-      />
-    </inertial>
-    <collision name='collision'>
-      <origin xyz="0 0 0" rpy=" 0 0 0"/>
-      <geometry>
-        <box size="0.05 0.05 0.05"/>
-      </geometry>
-    </collision>
-    <visual name='camera_visual'>
-      <origin xyz="0 0 0" rpy="0 0 0"/>
-      <geometry>
-        <box size="0.05 0.05 0.05"/>
-      </geometry>
-    </visual>
-  </link>
-  <joint type="fixed" name="camera_joint">
-    <origin xyz="0.2 0 0" rpy="0 0 0"/>
-    <child link="camera"/>
-    <parent link="chassis"/>
-    <axis xyz="0 1 0" rpy="0 0 0"/>
-    <limit effort="10000" velocity="1000"/>
-    <dynamics damping="1.0" friction="1.0"/>
-  </joint>
-	<!--	lidar-->
-	<link name='hokuyo'>
-    <pose>0 0 0 0 0 0</pose>
-    <inertial>
-      <mass value="1e-5"/>
-      <origin xyz="0.0 0 0" rpy="0.0 0 0"/>
-      <inertia
-          ixx="1e-6" ixy="0" ixz="0"
-          iyy="1e-6" iyz="0"
-          izz="1e-6"
-      />
-    </inertial>
-    <collision name='collision'>
-      <origin xyz="0 0 0" rpy=" 0 0 0"/>
-      <geometry>
-        <box size="0.1 0.1 0.1"/>
-      </geometry>
-    </collision>
-    <visual name='hokuyo_visual'>
-      <origin xyz="0 0 0" rpy="0 0 0"/>
-      <geometry>
-        <mesh filename="package://my_robot/meshes/hokuyo.dae"/>
-      </geometry>
-    </visual>
-  </link>
-  <joint type="fixed" name="hokuyo_joint">
-    <origin xyz="0.14 0.0 0.08" rpy="0 0 0"/>
-    <child link="hokuyo"/>
-    <parent link="chassis"/>
-    <axis xyz="0 1 0" rpy="0 0 0"/>
-    <limit effort="10000" velocity="1000"/>
-    <dynamics damping="1.0" friction="1.0"/>
-  </joint>
-	<!--visuals -->
-	<gazebo reference="left_wheel">
-		<material>Gazebo/Indigo</material>
-	</gazebo>
-	<gazebo reference="right_wheel">
-		<material>Gazebo/Indigo</material>
-	</gazebo>
-	<gazebo reference="chassis">
-		<material>Gazebo/Wood</material>
-	</gazebo>
-	<gazebo reference="camera">
-		<material>Gazebo/Red</material>
-	</gazebo>
-	<gazebo reference="add_mass">
-		<material>Gazebo/Black</material>
-	</gazebo>
+<link name='left_wheel_back'>
+  <inertial>
+    <mass value="5.0"/>
+    <origin xyz="0.0 0 0" rpy=" 0 1.5707 1.5707"/>
+    <inertia
+        ixx="0.1" ixy="0" ixz="0"
+        iyy="0.1" iyz="0"
+        izz="0.1"
+    />
+  </inertial>
+  <collision name='left_wheel_back_collision'>
+    <origin xyz="0 0 0" rpy=" 0 1.5707 1.5707"/>
+    <geometry>
+      <cylinder radius=".08" length="0.044"/>
+    </geometry>
+  </collision>
+  <visual name='left_wheel_back_visual'>
+    <origin xyz="0 0 0" rpy=" 0 1.5707 1.5707"/>
+    <geometry>
+      <cylinder radius=".08" length="0.044"/>
+    </geometry>
+  </visual>
+</link>
+<link name='right_wheel_front'>
+  <inertial>
+    <mass value="5.0"/>
+    <origin xyz="0.0 0 0" rpy=" 0 1.5707 1.5707"/>
+    <inertia
+        ixx="0.1" ixy="0" ixz="0"
+        iyy="0.1" iyz="0"
+        izz="0.1"
+    />
+  </inertial>
+  <collision name='right_wheel_front_collision'>
+    <origin xyz="0 0 0" rpy=" 0 1.5707 1.5707"/>
+    <geometry>
+      <cylinder radius=".08" length="0.044"/>
+    </geometry>
+  </collision>
+  <visual name='right_wheel_front_visual'>
+    <origin xyz="0 0 0" rpy=" 0 1.5707 1.5707"/>
+    <geometry>
+      <cylinder radius=".08" length="0.044"/>
+    </geometry>
+  </visual>
+</link>
+<link name='right_wheel_back'>
+  <inertial>
+    <mass value="5.0"/>
+    <origin xyz="0.0 0 0" rpy=" 0 1.5707 1.5707"/>
+    <inertia
+        ixx="0.1" ixy="0" ixz="0"
+        iyy="0.1" iyz="0"
+        izz="0.1"
+    />
+  </inertial>
+  <collision name='right_wheel_back_collision'>
+    <origin xyz="0 0 0" rpy=" 0 1.5707 1.5707"/>
+    <geometry>
+      <cylinder radius=".08" length="0.044"/>
+    </geometry>
+  </collision>
+  <visual name='right_wheel_back_visual'>
+    <origin xyz="0 0 0" rpy=" 0 1.5707 1.5707"/>
+    <geometry>
+      <cylinder radius=".08" length="0.044"/>
+    </geometry>
+  </visual>
+</link>
+<link name='camera'>
+  <inertial>
+    <mass value="0.1"/>
+    <origin xyz="0.0 0 0" rpy=" 0 0 0"/>
+    <inertia
+        ixx="1e-6" ixy="0" ixz="0"
+        iyy="1e-6" iyz="0"
+        izz="1e-6"
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